File: couchmobile-control/_autosave-couchmobile-electrical.kicad_pcb (KiCad board)
At the start: 2 copper layers, 100 x 100 mm, 50 parts, among them J1 Power_In, J10 Motor1, J11 Motor2, J2 GPIO_NANO_1, J5 ESTOP_IRQ_EN, J6 BNO_COMM_CTRL, J7 Joystick, J8 Encoder1, J9 Encoder2, Q1 PMOS DGS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

Commit message: Added 5v to 3.3v line converters.
Parts:
- added Q2: Q_NMOS_GSD, Package_TO_SOT_SMD:SOT-23, F.Cu at (86.5, 62.5)
- added Q3: Q_NMOS_GSD, Package_TO_SOT_SMD:SOT-23, F.Cu at (91.2, 62.5)
- added R20: 10k, Resistor_SMD:R_0805_2012Metric_Pad1.15x1.40mm_HandSolder, F.Cu at (79.2, 56.2)
- added R21: 10k, Resistor_SMD:R_0805_2012Metric_Pad1.15x1.40mm_HandSolder, F.Cu at (84.2, 56.2)
- added R22: 10k, Resistor_SMD:R_0805_2012Metric_Pad1.15x1.40mm_HandSolder, F.Cu at (76.8, 56.2)
- added R23: 10k, Resistor_SMD:R_0805_2012Metric_Pad1.15x1.40mm_HandSolder, F.Cu at (81.8, 56.2)
Connections:
- U2 pad 4: /SDA -> /SDA_3V3
- U2 pad 5: /SCL -> /SCL_3V3
Routing:
- net +5V: track 286.4 -> 363.8 mm
- net /SDA_3V3: track 0.00 -> 34.8 mm, vias 0 -> 1
- net /SCL_3V3: track 0.00 -> 29.5 mm, vias 0 -> 1
- net /SDA: track 65.5 -> 70.6 mm
- net /SCL: track 68.0 -> 71.3 mm
