File: couchmobile-control/couchmobile-electrical.sch (KiCad schematic (older format))
At the start: 50 parts

Commit message: Finished nano gpio
Connections:
- net labels added: NANO_A1, NANO_A2, NANO_A3, NANO_A4, NANO_A5, NANO_A6, NANO_A7, NANO_D8
- no-connect marks 0 -> 1
Other:
- note added: "Joystick module"
- note added: "NANO GPIO"
- note removed: "TODO:\nWire up RF module\nConnect GPIO banks"
Changed lines of the file:
@@
 L Connector_Generic:Conn_02x08_Odd_Even J?
 U 1 1 5D42C5D8
-P 1350 5400
-F 0 "J?" H 1400 5917 50  0000 C CNN
-F 1 "GPIO_MEGA_1" H 1400 5826 50  0000 C CNN
-F 2 "" H 1350 5400 50  0001 C CNN
-F 3 "~" H 1350 5400 50  0001 C CNN
-	1    1350 5400
+P 1350 5900
+F 0 "J?" H 1400 6417 50  0000 C CNN
+F 1 "GPIO_MEGA_1" H 1400 6326 50  0000 C CNN
+F 2 "" H 1350 5900 50  0001 C CNN
+F 3 "~" H 1350 5900 50  0001 C CNN
+	1    1350 5900
 	1    0    0    -1
 $EndComp
@@
 L Connector_Generic:Conn_02x08_Odd_Even J?
 U 1 1 5D42CA1E
-P 1350 6550
-F 0 "J?" H 1400 7067 50  0000 C CNN
-F 1 "GPIO_MEGA_2" H 1400 6976 50  0000 C CNN
-F 2 "" H 1350 6550 50  0001 C CNN
-F 3 "~" H 1350 6550 50  0001 C CNN
-	1    1350 6550
+P 1350 7050
+F 0 "J?" H 1400 7567 50  0000 C CNN
+F 1 "GPIO_MEGA_2" H 1400 7476 50  0000 C CNN
+F 2 "" H 1350 7050 50  0001 C CNN
+F 3 "~" H 1350 7050 50  0001 C CNN
+	1    1350 7050
 	1    0    0    -1
 $EndComp
@@
 L Connector_Generic:Conn_02x08_Odd_Even J?
 U 1 1 5D42E605
-P 1350 4250
-F 0 "J?" H 1400 4767 50  0000 C CNN
-F 1 "GPIO_NANO_1" H 1400 4676 50  0000 C CNN
-F 2 "" H 1350 4250 50  0001 C CNN
-F 3 "~" H 1350 4250 50  0001 C CNN
-	1    1350 4250
+P 1350 4400
+F 0 "J?" H 1400 4917 50  0000 C CNN
+F 1 "GPIO_NANO_1" H 1400 4826 50  0000 C CNN
+F 2 "" H 1350 4400 50  0001 C CNN
+F 3 "~" H 1350 4400 50  0001 C CNN
+	1    1350 4400
 	1    0    0    -1
 $EndComp
@@
 L RF:NRF24L01_Breakout U?
 U 1 1 5D463734
-P 3700 8950
-F 0 "U?" H 4178 8928 50  0000 L CNN
-F 1 "NRF24L01_Breakout" H 4178 8837 50  0000 L CNN
-F 2 "RF_Module:nRF24L01_Breakout" H 3850 9550 50  0001 L CIN
-F 3 "http://www.nordicsemi.com/eng/content/download/2730/34105/file/nRF24L01_Product_Specification_v2_0.pdf" H 3700 8850 50  0001 C CNN
-	1    3700 8950
+P 4200 9100
+F 0 "U?" H 4678 9078 50  0000 L CNN
+F 1 "NRF24L01_Breakout" H 4678 8987 50  0000 L CNN
+F 2 "RF_Module:nRF24L01_Breakout" H 4350 9700 50  0001 L CIN
+F 3 "http://www.nordicsemi.com/eng/content/download/2730/34105/file/nRF24L01_Product_Specification_v2_0.pdf" H 4200 9000 50  0001 C CNN
+	1    4200 9100
 	1    0    0    -1
 $EndComp
@@
 Text Notes 3850 2150 0    50   ~ 0
 ESTOP backup signal to control transistors
-Text Notes 11300 7850 0    50   ~ 0
-TODO:\nWire up RF module\nConnect GPIO banks
 $Comp
 L Device:R_Small R?
@@
 Text Label 14350 9050 0    50   ~ 0
 3V3
-Text Label 1150 5100 2    50   ~ 0
+Text Label 1150 5600 2    50   ~ 0
 5V
+Text Label 1150 6300 2    50   ~ 0
+3V3
+Text Label 1650 6300 0    50   ~ 0
+GND
+Text Label 1650 5600 0    50   ~ 0
+GND
+Text Label 1150 5700 2    50   ~ 0
+MEGA_RX0
+Text Label 1650 5700 0    50   ~ 0
+MEGA_TX0
+Text Label 1650 6200 0    50   ~ 0
+SCL
+Text Label 1150 6200 2    50   ~ 0
+SDA
 Text Label 1150 5800 2    50   ~ 0
-3V3
+MEGA_A6
+Text Label 1150 5900 2    50   ~ 0
+MEGA_A8
+Text Label 1150 6000 2    50   ~ 0
+MEGA_A10
+Text Label 1150 6100 2    50   ~ 0
+MEGA_A12
 Text Label 1650 5800 0    50   ~ 0
-GND
-Text Label 1650 5100 0    50   ~ 0
-GND
-Text Label 1150 5200 2    50   ~ 0
-MEGA_RX0
-Text Label 1650 5200 0    50   ~ 0
-MEGA_TX0
-Text Label 1650 5700 0    50   ~ 0
-SCL
-Text Label 1150 5700 2    50   ~ 0
-SDA
-Text Label 1150 5300 2    50   ~ 0
-MEGA_A6
-Text Label 1150 5400 2    50   ~ 0
-MEGA_A8
-Text Label 1150 5500 2    50   ~ 0
-MEGA_A10
-Text Label 1150 5600 2    50   ~ 0
-MEGA_A12
-Text Label 1650 5300 0    50   ~ 0
 MEGA_A7
-Text Label 1650 5400 0    50   ~ 0
+Text Label 1650 5900 0    50   ~ 0
 MEGA_A9
-Text Label 1650 5500 0    50   ~ 0
+Text Label 1650 6000 0    50   ~ 0
 MEGA_A11
-Text Label 1650 5600 0    50   ~ 0
+Text Label 1650 6100 0    50   ~ 0
 MEGA_A13
 Text Label 6450 1850 2    50   ~ 0
@@
 Text Label 6450 4450 2    50   ~ 0
 MEGA_A13
-Text Label 1150 6250 2    50   ~ 0
+Text Label 1150 6750 2    50   ~ 0
 5V
-Text Label 1650 6250 0    50   ~ 0
+Text Label 1650 6750 0    50   ~ 0
 GND
+Text Label 1150 7450 2    50   ~ 0
+3V3
+Text Label 1650 7450 0    50   ~ 0
+GND
+Text Label 1150 6850 2    50   ~ 0
+MEGA_A2
+Text Label 1650 6850 0    50   ~ 0
+MEGA_A3
 Text Label 1150 6950 2    50   ~ 0
-3V3
+MEGA_D32
+Text Label 1150 7050 2    50   ~ 0
+MEGA_D34
+Text Label 1150 7150 2    50   ~ 0
+MEGA_D36
+Text Label 1150 7250 2    50   ~ 0
+MEGA_D38
 Text Label 1650 6950 0    50   ~ 0
-GND
-Text Label 1150 6350 2    50   ~ 0
-MEGA_A2
-Text Label 1650 6350 0    50   ~ 0
-MEGA_A3
-Text Label 1150 6450 2    50   ~ 0
-MEGA_D32
-Text Label 1150 6550 2    50   ~ 0
-MEGA_D34
-Text Label 1150 6650 2    50   ~ 0
-MEGA_D36
-Text Label 1150 6750 2    50   ~ 0
-MEGA_D38
-Text Label 1650 6450 0    50   ~ 0
 MEGA_D33
-Text Label 1650 6550 0    50   ~ 0
+Text Label 1650 7050 0    50   ~ 0
 MEGA_D35
-Text Label 1650 6650 0    50   ~ 0
+Text Label 1650 7150 0    50   ~ 0
 MEGA_D37
-Text Label 1650 6750 0    50   ~ 0
+Text Label 1650 7250 0    50   ~ 0
 MEGA_D39
-Text Label 1150 6850 2    50   ~ 0
+Text Label 1150 7350 2    50   ~ 0
 SDA
-Text Label 1650 6850 0    50   ~ 0
+Text Label 1650 7350 0    50   ~ 0
 SCL
 Text Label 6450 3350 2    50   ~ 0
@@
 MEGA_D41
 Wire Notes Line
-	600  4800 2300 4800
-Wire Notes Line
-	2300 4800 2300 7200
-Wire Notes Line
-	2300 7200 600  7200
-Wire Notes Line
-	600  7200 600  4800
-Text Notes 700  7150 0    50   ~ 0
+	600  5300 2300 5300
+Wire Notes Line
+	2300 5300 2300 7700
+Wire Notes Line
+	2300 7700 600  7700
+Wire Notes Line
+	600  7700 600  5300
+Text Notes 700  7650 0    50   ~ 0
 MEGA GPIO and I2C pins
-Text Label 3200 8650 2    50   ~ 0
+Text Label 3700 8800 2    50   ~ 0
 ESTOP_MOSI
-Text Label 3200 8750 2    50   ~ 0
+Text Label 3700 8900 2    50   ~ 0
 ESTOP_MISO
-Text Label 3200 8850 2    50   ~ 0
+Text Label 3700 9000 2    50   ~ 0
 ESTOP_SCK
-Text Label 3200 8950 2    50   ~ 0
+Text Label 3700 9100 2    50   ~ 0
 ESTOP_CSN
-Text Label 3200 9150 2    50   ~ 0
+Text Label 3700 9300 2    50   ~ 0
 ESTOP_CE
 $Comp
 L power:+3V3 #PWR?
 U 1 1 5D590C79
-P 3700 8350
-F 0 "#PWR?" H 3700 8200 50  0001 C CNN
-F 1 "+3V3" H 3715 8523 50  0000 C CNN
-F 2 "" H 3700 8350 50  0001 C CNN
-F 3 "" H 3700 8350 50  0001 C CNN
-	1    3700 8350
+P 4200 8500
+F 0 "#PWR?" H 4200 8350 50  0001 C CNN
+F 1 "+3V3" H 4215 8673 50  0000 C CNN
+F 2 "" H 4200 8500 50  0001 C CNN
+F 3 "" H 4200 8500 50  0001 C CNN
+	1    4200 8500
 	1    0    0    -1
 $EndComp
@@
 L power:GND #PWR?
 U 1 1 5D590D0A
-P 3700 9550
-F 0 "#PWR?" H 3700 9300 50  0001 C CNN
-F 1 "GND" H 3705 9377 50  0000 C CNN
-F 2 "" H 3700 9550 50  0001 C CNN
-F 3 "" H 3700 9550 50  0001 C CNN
-	1    3700 9550
-	1    0    0    -1
-$EndComp
-Text Label 3200 9250 2    50   ~ 0
+P 4200 9700
+F 0 "#PWR?" H 4200 9450 50  0001 C CNN
+F 1 "GND" H 4205 9527 50  0000 C CNN
+F 2 "" H 4200 9700 50  0001 C CNN
+F 3 "" H 4200 9700 50  0001 C CNN
+	1    4200 9700
+	1    0    0    -1
+$EndComp
+Text Label 3700 9400 2    50   ~ 0
 ESTOP_IRQ
 Wire Notes Line
-	5050 8050 2600 8050
-Wire Notes Line
-	2600 8050 2600 10050
-Wire Notes Line
-	2600 10050 5050 10050
-Wire Notes Line
-	5050 10050 5050 8050
-Text Notes 2700 10000 0    50   ~ 0
+	5550 8200 3100 8200
+Wire Notes Line
+	3100 8200 3100 10200
+Wire Notes Line
+	3100 10200 5550 10200
+Wire Notes Line
+	5550 10200 5550 8200
+Text Notes 3200 10150 0    50   ~ 0
 ESTOP module
-Text Notes 3950 9600 0    50   ~ 0
+Text Notes 4450 9750 0    50   ~ 0
 Note: IRQ not in use
 Text Label 3350 2350 0    50   ~ 0
@@
 	1    0    0    -1
 $EndComp
-Text Label 1150 3950 2    50   ~ 0
+Text Label 1150 4100 2    50   ~ 0
 5V
-Text Label 1650 3950 0    50   ~ 0
+Text Label 1650 4100 0    50   ~ 0
 GND
-Text Label 1650 4650 0    50   ~ 0
+Text Label 1650 4800 0    50   ~ 0
 GND
-Text Label 1150 4650 2    50   ~ 0
+Text Label 1150 4800 2    50   ~ 0
 3V3
 Text Label 3350 1650 0    50   ~ 0
@@
 L Connector:Conn_01x02_Male J?
 U 1 1 5D5A27D7
-P 2800 9550
-F 0 "J?" H 2906 9728 50  0000 C CNN
-F 1 "ESTOP_IRQ_EN" H 2906 9637 50  0000 C CNN
-F 2 "" H 2800 9550 50  0001 C CNN
-F 3 "~" H 2800 9550 50  0001 C CNN
-	1    2800 9550
-	1    0    0    -1
-$EndComp
-Wire Wire Line
-	3200 9250 3150 9250
-Wire Wire Line
-	3150 9250 3150 9550
-Text Label 3100 9650 0    50   ~ 0
+P 3300 9700
+F 0 "J?" H 3406 9878 50  0000 C CNN
+F 1 "ESTOP_IRQ_EN" H 3406 9787 50  0000 C CNN
+F 2 "" H 3300 9700 50  0001 C CNN
+F 3 "~" H 3300 9700 50  0001 C CNN
+	1    3300 9700
+	1    0    0    -1
+$EndComp
+Wire Wire Line
+	3700 9400 3650 9400
+Wire Wire Line
+	3650 9400 3650 9700
+Text Label 3600 9800 0    50   ~ 0
 NANO_INT0
 Wire Wire Line
-	3000 9650 3100 9650
-Wire Wire Line
-	3000 9550 3150 9550
+	3500 9800 3600 9800
+Wire Wire Line
+	3500 9700 3650 9700
+Text Label 750  2050 2    50   ~ 0
+NANO_A7
+Text Label 750  2150 2    50   ~ 0
+NANO_A6
+Text Label 750  2250 2    50   ~ 0
+NANO_A5
+Text Label 750  2350 2    50   ~ 0
+NANO_A4
+Text Label 750  2450 2    50   ~ 0
+NANO_A3
+Text Label 750  2550 2    50   ~ 0
+NANO_A2
+Text Label 750  2650 2    50   ~ 0
+NANO_A1
+Text Label 1150 4200 2    50   ~ 0
+NANO_A7
+Text Label 1650 4200 0    50   ~ 0
+NANO_A6
+Text Label 1650 4300 0    50   ~ 0
+NANO_A4
+Text Label 1650 4400 0    50   ~ 0
+NANO_A2
+Text Label 1150 4300 2    50   ~ 0
+NANO_A5
+Text Label 1150 4400 2    50   ~ 0
+NANO_A3
+Text Label 1150 4500 2    50   ~ 0
+NANO_A1
+Text Label 3350 2250 0    50   ~ 0
+NANO_D8
+Text Label 1650 4500 0    50   ~ 0
+NANO_D8
+Text Label 1150 4600 2    50   ~ 0
+ESTOP_ON
+Text Label 1650 4600 0    50   ~ 0
+ESTOP_HS
+Text Label 1150 4700 2    50   ~ 0
+NANO_RX
+Text Label 1650 4700 0    50   ~ 0
+NANO_TX
+Wire Notes Line
+	600  3800 2300 3800
+Wire Notes Line
+	2300 3800 2300 5150
+Wire Notes Line
+	2300 5150 600  5150
+Wire Notes Line
+	600  5150 600  3800
+Text Notes 700  5100 0    50   ~ 0
+NANO GPIO
+NoConn ~ 13050 1450
+Wire Notes Line
+	11100 1550 13850 1550
+Wire Notes Line
+	13850 1550 13850 800
+Wire Notes Line
+	13850 800  11100 800
+Wire Notes Line
+	11100 800  11100 1550
+Text Notes 11200 1500 0    50   ~ 0
+Joystick module
 $EndSCHEMATC

Commit message: Finished wiring up schematic; DRC passed. ALso added in the AND gates
Parts:
- removed SW?: SW_SP3T, symbol Switch:SW_SP3T
- added Q1: PMOS DGS, Package_SO:SO-8_5.3x6.2mm_P1.27mm, symbol Device:Q_PMOS_DGS
- added SW3: User Switch, couch-switches:MTS_3_pin_toggle_switch, symbol Switch:SW_SPDT_MSM
- added U3: 74LS08, Package_DIP:DIP-14_W7.62mm, symbol 74xx:74LS08
- D1, D2, D3, D4, D5, D6, D7, D8, D9: renamed from D?; footprint (none) -> LED_SMD:LED_0805_2012Metric_Pad1.15x1.40mm_HandSolder
- J1: renamed from J?; footprint (none) -> TerminalBlock:TerminalBlock_bornier-2_P5.08mm
- J10, J11: renamed from J?; footprint (none) -> Connector_PinHeader_2.54mm:PinHeader_1x03_P2.54mm_Vertical
- J2, J3, J4: renamed from J?; footprint (none) -> Connector_PinHeader_2.54mm:PinHeader_2x08_P2.54mm_Vertical
- J5: renamed from J?; footprint (none) -> Connector_PinHeader_2.54mm:PinHeader_1x02_P2.54mm_Vertical
- J6: renamed from J?; footprint (none) -> Connector_PinHeader_2.54mm:PinHeader_2x03_P2.54mm_Vertical
- J7, J8, J9: renamed from J?; footprint (none) -> Connector_PinHeader_2.54mm:PinHeader_1x06_P2.54mm_Vertical
- MH1, MH2, MH3, MH4: renamed from MH?; footprint (none) -> MountingHole:MountingHole_3.2mm_M3_ISO7380
- R1, R10, R11, R12, R13, R14, R15, R16, R17, R18, R19, R2, R3, R4, R5, R6, R7, R8, R9: renamed from R?; footprint (none) -> Resistor_SMD:R_0805_2012Metric_Pad1.15x1.40mm_HandSolder
- SW1, SW2: renamed from SW?; footprint (none) -> Button_Switch_THT:SW_TH_Tactile_Omron_B3F-10xx
- U2: renamed from U?; footprint (none) -> BNO080:BNO080
- XA1: renamed from XA?; footprint (none) -> Arduino:Arduino_Nano_Socket
- XA2: renamed from XA?; footprint (none) -> Arduino:Arduino_Mega2560_Shield
- gave numbers to parts that had none: 1
Connections:
- net labels added: M1_OUT, M2_OUT
- net labels removed: IMU_INT, MEGA_D40, MEGA_D41
- wire segments 151 -> 170
- no-connect marks 1 -> 37

Commit message: Made and added so8 package for pfet
Parts:
- Q1: footprint Package_SO:SO-8_5.3x6.2mm_P1.27mm -> couch-packages:SO-8_DGS
Changed lines of the file:
@@
 F 0 "Q1" V 2393 850 50  0000 C CNN
 F 1 "PMOS DGS" V 2302 850 50  0000 C CNN
-F 2 "Package_SO:SO-8_5.3x6.2mm_P1.27mm" H 2250 950 50  0001 C CNN
+F 2 "couch-packages:SO-8_DGS" H 2250 950 50  0001 C CNN
 F 3 "~" H 2050 850 50  0001 C CNN
 	1    2050 850

Commit message: Added 5v to 3.3v line converters.
Parts:
- added Q2, Q3: Q_NMOS_GSD, Package_TO_SOT_SMD:SOT-23, symbol Device:Q_NMOS_GSD
- added R20, R21, R22, R23: 10k, Resistor_SMD:R_0805_2012Metric_Pad1.15x1.40mm_HandSolder, symbol Device:R_Small
Connections:
- net labels added: SCL_3V3, SDA_3V3
- wire segments 170 -> 195
Changed lines of the file:
@@
 	7050 9550 7050 9600
 Text Label 7500 9750 2    50   ~ 0
-SDA
+SDA_3V3
 Text Label 7500 9850 2    50   ~ 0
-SCL
+SCL_3V3
 Text Label 8400 9650 0    50   ~ 0
 MISO
@@
 L Mechanical:MountingHole MH1
 U 1 1 5D59A92A
-P 10900 8950
-F 0 "MH1" H 11000 8996 50  0000 L CNN
-F 1 "MountingHole" H 11000 8905 50  0000 L CNN
-F 2 "MountingHole:MountingHole_3.2mm_M3_ISO7380" H 10900 8950 50  0001 C CNN
-F 3 "~" H 10900 8950 50  0001 C CNN
-	1    10900 8950
+P 14850 6950
+F 0 "MH1" H 14950 6996 50  0000 L CNN
+F 1 "MountingHole" H 14950 6905 50  0000 L CNN
+F 2 "MountingHole:MountingHole_3.2mm_M3_ISO7380" H 14850 6950 50  0001 C CNN
+F 3 "~" H 14850 6950 50  0001 C CNN
+	1    14850 6950
 	1    0    0    -1
 $EndComp
@@
 L Mechanical:MountingHole MH2
 U 1 1 5D59AA96
-P 10900 9200
-F 0 "MH2" H 11000 9246 50  0000 L CNN
-F 1 "MountingHole" H 11000 9155 50  0000 L CNN
-F 2 "MountingHole:MountingHole_3.2mm_M3_ISO7380" H 10900 9200 50  0001 C CNN
-F 3 "~" H 10900 9200 50  0001 C CNN
-	1    10900 9200
+P 14850 7200
+F 0 "MH2" H 14950 7246 50  0000 L CNN
+F 1 "MountingHole" H 14950 7155 50  0000 L CNN
+F 2 "MountingHole:MountingHole_3.2mm_M3_ISO7380" H 14850 7200 50  0001 C CNN
+F 3 "~" H 14850 7200 50  0001 C CNN
+	1    14850 7200
 	1    0    0    -1
 $EndComp
@@
 L Mechanical:MountingHole MH3
 U 1 1 5D59ABDD
-P 10900 9450
-F 0 "MH3" H 11000 9496 50  0000 L CNN
-F 1 "MountingHole" H 11000 9405 50  0000 L CNN
-F 2 "MountingHole:MountingHole_3.2mm_M3_ISO7380" H 10900 9450 50  0001 C CNN
-F 3 "~" H 10900 9450 50  0001 C CNN
-	1    10900 9450
+P 14850 7450
+F 0 "MH3" H 14950 7496 50  0000 L CNN
+F 1 "MountingHole" H 14950 7405 50  0000 L CNN
+F 2 "MountingHole:MountingHole_3.2mm_M3_ISO7380" H 14850 7450 50  0001 C CNN
+F 3 "~" H 14850 7450 50  0001 C CNN
+	1    14850 7450
 	1    0    0    -1
 $EndComp
@@
 L Mechanical:MountingHole MH4
 U 1 1 5D59ABE4
-P 10900 9700
-F 0 "MH4" H 11000 9746 50  0000 L CNN
-F 1 "MountingHole" H 11000 9655 50  0000 L CNN
-F 2 "MountingHole:MountingHole_3.2mm_M3_ISO7380" H 10900 9700 50  0001 C CNN
-F 3 "~" H 10900 9700 50  0001 C CNN
-	1    10900 9700
+P 14850 7700
+F 0 "MH4" H 14950 7746 50  0000 L CNN
+F 1 "MountingHole" H 14950 7655 50  0000 L CNN
+F 2 "MountingHole:MountingHole_3.2mm_M3_ISO7380" H 14850 7700 50  0001 C CNN
+F 3 "~" H 14850 7700 50  0001 C CNN
+	1    14850 7700
 	1    0    0    -1
 $EndComp
@@
 Text Label 9050 4850 0    50   ~ 0
 JOYSTICK_SW
+Wire Wire Line
+	10800 9250 11800 9250
+Wire Wire Line
+	11800 9250 11800 9100
+Wire Wire Line
+	10800 9250 10650 9250
+Connection ~ 10800 9250
+$Comp
+L power:+3V3 #PWR0146
+U 1 1 5D8B8B2D
+P 10650 9200
+F 0 "#PWR0146" H 10650 9050 50  0001 C CNN
+F 1 "+3V3" H 10665 9373 50  0000 C CNN
+F 2 "" H 10650 9200 50  0001 C CNN
+F 3 "" H 10650 9200 50  0001 C CNN
+	1    10650 9200
+	1    0    0    -1
+$EndComp
+Wire Wire Line
+	10650 9250 10650 9200
+Wire Wire Line
+	10800 8650 10800 9250
+Text Label 9800 8350 2    50   ~ 0
+SCL
+Text Label 9800 8800 2    50   ~ 0
+SDA
+$Comp
+L Device:R_Small R23
+U 1 1 5D8ECAD5
+P 12400 9050
+F 0 "R23" H 12459 9096 50  0000 L CNN
+F 1 "10k" H 12459 9005 50  0000 L CNN
+F 2 "Resistor_SMD:R_0805_2012Metric_Pad1.15x1.40mm_HandSolder" H 12400 9050 50  0001 C CNN
+F 3 "~" H 12400 9050 50  0001 C CNN
+	1    12400 9050
+	1    0    0    -1
+$EndComp
+Wire Wire Line
+	12000 8800 12400 8800
+Wire Wire Line
+	12400 9150 12400 9250
+Connection ~ 11800 9250
+Wire Wire Line
+	12400 8950 12400 8800
+Connection ~ 12400 8800
+Wire Wire Line
+	12400 8800 12500 8800
+$Comp
+L Device:R_Small R21
+U 1 1 5D946483
+P 10350 8050
+F 0 "R21" H 10409 8096 50  0000 L CNN
+F 1 "10k" H 10409 8005 50  0000 L CNN
+F 2 "Resistor_SMD:R_0805_2012Metric_Pad1.15x1.40mm_HandSolder" H 10350 8050 50  0001 C CNN
+F 3 "~" H 10350 8050 50  0001 C CNN
+	1    10350 8050
+	1    0    0    -1
+$EndComp
+$Comp
+L Device:R_Small R20
+U 1 1 5D94651D
+P 10050 8050
+F 0 "R20" H 10109 8096 50  0000 L CNN
+F 1 "10k" H 10109 8005 50  0000 L CNN
+F 2 "Resistor_SMD:R_0805_2012Metric_Pad1.15x1.40mm_HandSolder" H 10050 8050 50  0001 C CNN
+F 3 "~" H 10050 8050 50  0001 C CNN
+	1    10050 8050
+	1    0    0    -1
+$EndComp
+Wire Wire Line
+	11000 8350 12150 8350
+Wire Wire Line
+	11800 9250 12150 9250
+$Comp
+L Device:R_Small R22
+U 1 1 5D946741
+P 12150 9050
+F 0 "R22" H 12209 9096 50  0000 L CNN
+F 1 "10k" H 12209 9005 50  0000 L CNN
+F 2 "Resistor_SMD:R_0805_2012Metric_Pad1.15x1.40mm_HandSolder" H 12150 9050 50  0001 C CNN
+F 3 "~" H 12150 9050 50  0001 C CNN
+	1    12150 9050
+	1    0    0    -1
+$EndComp
+Wire Wire Line
+	12150 9150 12150 9250
+Connection ~ 12150 9250
+Wire Wire Line
+	12150 9250 12400 9250
+Wire Wire Line
+	12150 8950 12150 8350
+Connection ~ 12150 8350
+Wire Wire Line
+	12150 8350 12500 8350
+Wire Wire Line
+	10350 8150 10350 8800
+Wire Wire Line
+	10350 8800 11600 8800
+Wire Wire Line
+	10050 8350 10050 8150
+Wire Wire Line
+	10050 8350 10600 8350
+Wire Wire Line
+	10350 7950 10350 7850
+Wire Wire Line
+	10350 7850 10050 7850
+Wire Wire Line
+	10050 7850 10050 7950
+$Comp
+L power:+5V #PWR0147
+U 1 1 5D9AE183
+P 10050 7750
+F 0 "#PWR0147" H 10050 7600 50  0001 C CNN
+F 1 "+5V" H 10065 7923 50  0000 C CNN
+F 2 "" H 10050 7750 50  0001 C CNN
+F 3 "" H 10050 7750 50  0001 C CNN
+	1    10050 7750
+	1    0    0    -1
+$EndComp
+Wire Wire Line
+	10050 7750 10050 7850
+Connection ~ 10050 7850
+Wire Wire Line
+	9800 8800 10350 8800
+Connection ~ 10350 8800
+Wire Wire Line
+	10050 8350 9800 8350
+Connection ~ 10050 8350
+Text Label 12500 8350 0    50   ~ 0
+SCL_3V3
+Text Label 12500 8800 0    50   ~ 0
+SDA_3V3
+$Comp
+L Device:Q_NMOS_GSD Q2
+U 1 1 5D9D33EE
+P 10800 8450
+F 0 "Q2" V 11143 8450 50  0000 C CNN
+F 1 "Q_NMOS_GSD" V 11052 8450 50  0000 C CNN
+F 2 "Package_TO_SOT_SMD:SOT-23" H 11000 8550 50  0001 C CNN
+F 3 "~" H 10800 8450 50  0001 C CNN
+	1    10800 8450
+	0    -1   -1   0
+$EndComp
+$Comp
+L Device:Q_NMOS_GSD Q3
+U 1 1 5D9D3554
+P 11800 8900
+F 0 "Q3" V 12143 8900 50  0000 C CNN
+F 1 "Q_NMOS_GSD" V 12052 8900 50  0000 C CNN
+F 2 "Package_TO_SOT_SMD:SOT-23" H 12000 9000 50  0001 C CNN
+F 3 "~" H 11800 8900 50  0001 C CNN
+	1    11800 8900
+	0    -1   -1   0
+$EndComp
 $EndSCHEMATC

Commit message: Changed some resistor values. Generated BOM.
Parts:
- Q2, Q3: value Q_NMOS_GSD -> BSS138; Purchase Link (none) -> https://www.digikey.com.au/product-detail/en/on-semiconduct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
- R6, R7: value 10k -> 2.2k
- U3: Supplier Link (none) -> https://www.digikey.com/product-detail/en/texas-instruments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
Changed lines of the file:
@@
 P 12350 5700
 F 0 "R6" V 12546 5700 50  0000 C CNN
-F 1 "10k" V 12455 5700 50  0000 C CNN
+F 1 "2.2k" V 12455 5700 50  0000 C CNN
 F 2 "Resistor_SMD:R_0805_2012Metric_Pad1.15x1.40mm_HandSolder" H 12350 5700 50  0001 C CNN
 F 3 "~" H 12350 5700 50  0001 C CNN
@@
 P 12350 6050
 F 0 "R7" V 12546 6050 50  0000 C CNN
-F 1 "10k" V 12455 6050 50  0000 C CNN
+F 1 "2.2k" V 12455 6050 50  0000 C CNN
 F 2 "Resistor_SMD:R_0805_2012Metric_Pad1.15x1.40mm_HandSolder" H 12350 6050 50  0001 C CNN
 F 3 "~" H 12350 6050 50  0001 C CNN
@@
 F 2 "Package_DIP:DIP-14_W7.62mm" H 10350 3150 50  0001 C CNN
 F 3 "http://www.ti.com/lit/gpn/sn74LS08" H 10350 3150 50  0001 C CNN
+F 4 "https://www.digikey.com/product-detail/en/texas-instruments/SN74HC08N/296-1570-5-ND/277216" V 10350 3150 50  0001 C CNN "Supplier Link"
 	5    10350 3150
 	0    -1   -1   0
@@
 P 10800 8450
 F 0 "Q2" V 11143 8450 50  0000 C CNN
-F 1 "Q_NMOS_GSD" V 11052 8450 50  0000 C CNN
+F 1 "BSS138" V 11052 8450 50  0000 C CNN
 F 2 "Package_TO_SOT_SMD:SOT-23" H 11000 8550 50  0001 C CNN
-F 3 "~" H 10800 8450 50  0001 C CNN
+F 3 "https://www.onsemi.com/pub/Collateral/BSS138LT1-D.PDF" H 10800 8450 50  0001 C CNN
+F 4 "https://www.digikey.com.au/product-detail/en/on-semiconductor/BSS138LT3G/BSS138LT3GOSCT-ND/2120566" V 10800 8450 50  0001 C CNN "Purchase Link"
 	1    10800 8450
 	0    -1   -1   0
@@
 P 11800 8900
 F 0 "Q3" V 12143 8900 50  0000 C CNN
-F 1 "Q_NMOS_GSD" V 12052 8900 50  0000 C CNN
+F 1 "BSS138" V 12052 8900 50  0000 C CNN
 F 2 "Package_TO_SOT_SMD:SOT-23" H 12000 9000 50  0001 C CNN
-F 3 "~" H 11800 8900 50  0001 C CNN
+F 3 "https://www.onsemi.com/pub/Collateral/BSS138LT1-D.PDF" H 11800 8900 50  0001 C CNN
+F 4 "https://www.digikey.com.au/product-detail/en/on-semiconductor/BSS138LT3G/BSS138LT3GOSCT-ND/2120566" V 11800 8900 50  0001 C CNN "Purchase Link"
 	1    11800 8900
 	0    -1   -1   0
