File: couchmobile-control/rev1/couchmobile-electrical.sch (KiCad schematic (older format))
At the start: 58 parts, among them J1 Power_In, J10 Motor1, J11 Motor2, J2 GPIO_NANO_1, J3 GPIO_MEGA_1, J4 GPIO_MEGA_2, J5 ESTOP_IRQ_EN, J6 BNO_COMM_CTRL, J7 Conn_02x04_Top_Bottom, J8 Encoder1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

Commit message: Added in label to control panel
Connections:
- no-connect marks 39 -> 41
Changed lines of the file:
@@
 NoConn ~ 8400 9650
 NoConn ~ 8400 9750
+NoConn ~ 13250 1050
+NoConn ~ 13250 1150
 $EndSCHEMATC
