File: control pad/control pad.kicad_pcb (KiCad board)
At the start: 2 copper layers, 81.3 x 91.4 mm, 16 parts, among them J1 IDC CONNECTOR 02x04, J2 Conn_01x02, U1 RC1602A, U2 analogstick

Commit message: finished v0 of control pad pcb
Parts:
- added D5: LED, Diode_SMD:D_0805_2012Metric_Pad1.15x1.40mm_HandSolder, F.Cu at (153.4, 121.7)
- added R8: 330, Resistor_SMD:R_0805_2012Metric_Pad1.15x1.40mm_HandSolder, F.Cu at (148.3, 121.7)
- D1, D2, D3, D4, R4, R5, R6, R7, U2: moved to F.Cu
- moved D1 32.8 mm to (153.4, 131.8)
- moved R4 32.8 mm to (148.3, 131.8)
- moved D2 27.7 mm to (153.4, 129.3)
- moved R5 27.7 mm to (148.3, 129.3)
- moved R6 22.6 mm to (148.3, 126.7)
- moved D3 22.6 mm to (153.4, 126.7)
- moved R7 17.6 mm to (148.3, 124.2)
- moved D4 17.6 mm to (153.4, 124.2)
- moved R3 1.52 mm to (188.0, 90.4)
- turned U2 to 270 degrees
Routing:
- net GND: track 138.8 -> 117.3 mm
- net Net-(A1-Pad15): track 0.00 -> 16.6 mm
- net 5V: track 47.7 -> 38.5 mm
- net Net-(A1-Pad14): track 14.8 -> 21.0 mm
- net Net-(A1-Pad13): track 18.4 -> 23.7 mm
- net Net-(A1-Pad12): track 22.0 -> 27.3 mm
- net Net-(A1-Pad11): track 25.5 -> 30.9 mm
- net Net-(D5-Pad1): track 0.00 -> 3.02 mm
- net Net-(R3-Pad1): track 2.78 -> 4.80 mm
Other:
- board text added: "Control Panel Board v0 By Vignaraj Mahapatra"
- board text added: "GND"
- board text added: "KEY"
- board text added: "PWR"
- board text added: "RX"
- board text added: "STOP"
- board text added: "TX"

Commit message: Updated labels on pcb revision 3
Other:
- board text added: "AUTO"
- board text removed: "KEY"
Changed lines of the file:
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@@
     (effects (font (size 1 1) (thickness 0.15)) (justify left))
   )
-  (gr_text KEY (at 156.972 124.206) (layer F.SilkS)
+  (gr_text AUTO (at 157.48 126.746) (layer F.SilkS)
     (effects (font (size 1 1) (thickness 0.15)))
   )
-  (gr_text "STOP\n" (at 157.48 126.746) (layer F.SilkS)
+  (gr_text "STOP\n" (at 157.48 124.206) (layer F.SilkS)
     (effects (font (size 1 1) (thickness 0.15)))
   )
-  (gr_text TX (at 156.718 129.286) (layer F.SilkS)
+  (gr_text TX (at 156.464 131.826) (layer F.SilkS)
     (effects (font (size 1 1) (thickness 0.15)))
   )
-  (gr_text RX (at 156.718 131.826) (layer F.SilkS)
+  (gr_text RX (at 156.464 129.286) (layer F.SilkS)
     (effects (font (size 1 1) (thickness 0.15)))
   )
